Commit message: Real-hardware kinematic fix + first end-to-end real motion + diagnostic tooling
Two-line URDF fix that resolves the URDF/cabinet kinematic mismatch:

  ur_macro.xacro line 350:  rpy "0 0 pi" reverted to rpy "0 0 0"
  ur_macro.xacro line 364:  axis xyz "0 0 -1" reverted to axis xyz "0 0 1"

The upstream 180-degree base_link to base_link_inertia yaw and my earlier
shoulder_pan axis flip cancelled out at HOME by symmetry, but together
caused a 180-degree-class mirror at any non-HOME pose. With both reverted,
URDF FK matches cabinet RTDE TCP within 0.4 mm at HOME AND at an extreme
freedrive pose [all 6 joints displaced] - verified with the new
tcp_compare.py read-only diagnostic.

This session's results:
  - First real-hardware motion ever under ROS 2 control
  - External Control URCap installed and URP configured on cabinet
  - Windows Firewall inbound rule for 50001-50004 from cabinet
  - URDF kinematic mismatch root-caused via fk_experiment.py
    [tests 4 hypotheses against measured RTDE; only B matches everywhere]
  - Fix applied and verified at 0.4 mm precision
  - First non-symmetric Cartesian motion succeeded on real hardware
    [3 LIN moves correctly reached world-frame targets]
  - Identified secondary LIFT IK issue [collision/singularity, not kinematics]

Known issues to follow up:
  - LIFT IK fails at TCP X=0.823 Y=0.473 Z=0.500 - hypotheses in SESSION_HANDOFF
  - URScript-via-topic gripper not closing [URP preamble issue]
  - Sim play_pickplace LIFT regression mirrors real LIFT [same root cause]
  - RTDE 500 Hz hardcoded in driver; would need patch to expose as param

Co-Authored-By: Claude Opus 4.7 <noreply@anthropic.com>

File: src/Universal_Robots_ROS2_Description/urdf/ur10e_rg6.urdf.xacro (robot description, xacro)
@@ -5,4 +5,19 @@
   <xacro:arg name="fake_sensor_commands" default="false"/>
   <xacro:arg name="robot_ip"             default="0.0.0.0"/>
+  <!-- Real-hardware args forwarded from ur_control.launch.py. Without these
+       declared at the top level, xacro silently drops them and ur_macro's
+       defaults ('to_be_filled_by_ur_robot_driver') reach the C++ driver,
+       which aborts on file open (2026-05-26 incident, wiki/known_bugs). -->
+  <xacro:arg name="headless_mode"          default="false"/>
+  <xacro:arg name="script_filename"        default=""/>
+  <xacro:arg name="output_recipe_filename" default=""/>
+  <xacro:arg name="input_recipe_filename"  default=""/>
+  <xacro:arg name="reverse_ip"             default="0.0.0.0"/>
+  <xacro:arg name="reverse_port"           default="50001"/>
+  <xacro:arg name="script_sender_port"     default="50002"/>
+  <xacro:arg name="trajectory_port"        default="50003"/>
+  <xacro:arg name="script_command_port"    default="50004"/>
+  <xacro:arg name="non_blocking_read"      default="true"/>
+  <xacro:arg name="keep_alive_count"       default="2"/>
   <!-- ====================================================== -->
   <!-- Include UR10e macros and ROS2 control                  -->
@@ -61,4 +76,15 @@
       fake_sensor_commands="$(arg fake_sensor_commands)"
       robot_ip="$(arg robot_ip)"
+      headless_mode="$(arg headless_mode)"
+      script_filename="$(arg script_filename)"
+      output_recipe_filename="$(arg output_recipe_filename)"
+      input_recipe_filename="$(arg input_recipe_filename)"
+      reverse_ip="$(arg reverse_ip)"
+      reverse_port="$(arg reverse_port)"
+      script_sender_port="$(arg script_sender_port)"
+      trajectory_port="$(arg trajectory_port)"
+      script_command_port="$(arg script_command_port)"
+      non_blocking_read="$(arg non_blocking_read)"
+      keep_alive_count="$(arg keep_alive_count)"
       generate_ros2_control_tag="true">
     <origin xyz="0 0 0" rpy="0 0 0"/>
@@ -114,5 +140,10 @@
     <origin xyz="0 0 0.051" rpy="0 0 0"/>
   </joint>
-  <!-- 3. Grasp frame (TCP) — 190 mm down the gripper Z axis -->
+  <!-- 3. Grasp frame (TCP) — 228 mm down the gripper Z axis.
+       Calibrated 2026-05-26 against the real cabinet's set_tcp() offset:
+       at HOME the cabinet's RTDE-reported TCP Z (0.400 m) is 0.279 m below
+       URDF tool0 Z (0.679 m). Our chain has bracket(0) + body(0.051) +
+       grasp(?) = total 0.279 → grasp = 0.228 m. Previous value 0.190 m
+       under-estimated the gripper length by 38 mm. -->
   <link name="rg6_tcp">
     <visual>
@@ -124,5 +155,5 @@
     <parent link="rg6_body"/>
     <child link="rg6_tcp"/>
-    <origin xyz="0 0 0.19" rpy="0 0 0"/>
+    <origin xyz="0 0 0.228" rpy="0 0 0"/>
   </joint>
   <!-- 4. ee_link alias for MoveIt -->
@@ -243,11 +274,12 @@
   <!-- ====================================================== -->
   <ros2_control name="OnRobotRG6System" type="system">
+    <!-- LOCKED DECISION (wiki/decisions.md 2026-05-24): RG6 control on real
+         hardware uses Mechanism C (URScript topic via /urscript_interface/
+         script_command), NOT the onrobot_interface C++ plugin. The plugin
+         requires prefix/model params we don't pass and crashes on init.
+         Always use mock_components so the joint exists for state mirroring;
+         the real gripper is commanded outside ros2_control entirely. -->
     <hardware>
-      <xacro:if value="$(arg use_fake_hardware)">
-        <plugin>mock_components/GenericSystem</plugin>
-      </xacro:if>
-      <xacro:unless value="$(arg use_fake_hardware)">
-        <plugin>onrobot_interface::OnRobotHardwareInterface</plugin>
-      </xacro:unless>
+      <plugin>mock_components/GenericSystem</plugin>
     </hardware>
     <joint name="rg6_joint">
